File: ICCI-HW/USB.kicad_sch (KiCad schematic)
At the start: 9 parts

Commit message: usb PD started
Other:
- moved on the sheet: U?
Changed lines of the file:
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@@
     (effects (font (size 2.9972 2.9972) (thickness 0.5994) bold) (justify right bottom))
   )
-  (text "USB BC (Battery Charging)\nStandard coesistente con USB PD (Power Delivery)\nPermette di eccedere i 500mA in USB2.0 e 900mA in USB3.0\ned arrivare fino a 1.5A. NOTA: siccome i connettori USB\nsupportano fino a 5A, alcuni produttori alzano la corrente\nfino a livelli più alti (tipo i classici 2A).\nIl dispositivo caricatore si identifica come tale\nsegnalando l'assenza di dati nei segnali D+ e D- ponendo\nun resistore da meno di 200ohm tra D+ e D-.\nNon è possibile quindi eccedere i 500mA per USB2.0 ed\nutilizzar il trasferimento di dati simutaneamente.\nUSB BC da scartare perchè tensione massima è 5V ed è troppo\nbassa per caricare 2 Li-Ion in serie (senza usare DCDC).\n\nUSB C power delivery (NOTA: disponibile con connettore C) \nnon consente il trasferimento di dati \nsimultaneamente al PD.\nUna soluzione è quella di usare un comunissimo\nCP2102/CP2104 quando l'usb viene connessa ad un\ndispisitivo di comunicazione con Vbus=5V, mentre\nutilizzare un chip per USB PD quando l'usb è\ncollegato ad un dispositivo di ricarica PD.\nIn sostanza collegando un dispositivo di tipo PD\nil chip che gestisce la PD richiederà la tensione\ne la corrente volute (farà da sink) al dispositivo \nsource PD.\nQuando invece viene collegato un dispositivo USB\nnormale il chip che gestisce la USB utilizzerà le\nlinee di dato normalmente (USB2 o USB3 che sia) e \nil chip PD non interverrà."
-    (at 301.625 109.855 0)
+  (text "USB BC (Battery Charging)\nStandard coesistente con USB PD (Power Delivery)\nPermette di eccedere i 500mA in USB2.0 e 900mA in USB3.0\ned arrivare fino a 1.5A. NOTA: siccome i connettori USB\nsupportano fino a 5A, alcuni produttori alzano la corrente\nfino a livelli più alti (tipo i classici 2A).\nIl dispositivo caricatore si identifica come tale\nsegnalando l'assenza di dati nei segnali D+ e D- ponendo\nun resistore da meno di 200ohm tra D+ e D-.\nNon è possibile quindi eccedere i 500mA per USB2.0 ed\nutilizzar il trasferimento di dati simutaneamente.\nUSB BC da scartare perchè tensione massima è 5V ed è troppo\nbassa per caricare 2 Li-Ion in serie (senza usare DCDC).\n\nUSB C power delivery (NOTA: disponibile con connettore C) \nnon consente il trasferimento di dati \nsimultaneamente al PD.\nUna soluzione è quella di usare un comunissimo\nCP2102/CP2104 quando l'usb viene connessa ad un\ndispisitivo di comunicazione con Vbus=5V, mentre\nutilizzare un chip per USB PD quando l'usb è\ncollegato ad un dispositivo di ricarica PD.\nIn sostanza collegando un dispositivo di tipo PD\nil chip che gestisce la PD richiederà la tensione\ne la corrente volute (farà da sink) al dispositivo \nsource PD.\nQuando invece viene collegato un dispositivo USB\nnormale il chip che gestisce la USB utilizzerà le\nlinee di dato normalmente (USB2 o USB3 che sia) e \nil chip PD non interverrà.\n\nNOTA: vanno gestiti i vari casi:\n- USB 5V 100mA\n- USB 5V 500mA\n- USB BC 5V 1.5A\n- USB PD"
+    (at 182.88 132.08 0)
     (effects (font (size 2.032 2.032)) (justify left bottom))
   )
@@
     (pin "1")
   )
-  (symbol (lib_id "Interface_USB:CP2102N-Axx-xQFN28") (at 133.35 68.58 0) (unit 1)
+  (symbol (lib_id "Interface_USB:CP2102N-Axx-xQFN28") (at 36.195 117.475 0) (unit 1)
     (in_bom yes) (on_board yes) (fields_autoplaced)
-    (property "Reference" "U?" (id 0) (at 135.3694 102.235 0)
+    (property "Reference" "U?" (id 0) (at 38.2144 151.13 0)
       (effects (font (size 1.27 1.27)) (justify left))
     )
-    (property "Value" "CP2102N-Axx-xQFN28" (id 1) (at 135.3694 104.775 0)
+    (property "Value" "CP2102N-Axx-xQFN28" (id 1) (at 38.2144 153.67 0)
       (effects (font (size 1.27 1.27)) (justify left))
     )
-    (property "Footprint" "Package_DFN_QFN:QFN-28-1EP_5x5mm_P0.5mm_EP3.35x3.35mm" (id 2) (at 166.37 100.33 0)
+    (property "Footprint" "Package_DFN_QFN:QFN-28-1EP_5x5mm_P0.5mm_EP3.35x3.35mm" (id 2) (at 69.215 149.225 0)
       (effects (font (size 1.27 1.27)) hide)
     )
-    (property "Datasheet" "https://www.silabs.com/documents/public/data-sheets/cp2102n-datasheet.pdf" (id 3) (at 134.62 87.63 0)
+    (property "Datasheet" "https://www.silabs.com/documents/public/data-sheets/cp2102n-datasheet.pdf" (id 3) (at 37.465 136.525 0)
       (effects (font (size 1.27 1.27)) hide)
     )
@@
     (pin "9")
   )
-  (symbol (lib_id "ICCI-LIB:UPD301B{slash}C") (at 202.565 40.005 0) (unit 1)
+  (symbol (lib_id "ICCI-LIB:UPD301B{slash}C") (at 114.3 95.25 0) (unit 1)
     (in_bom yes) (on_board yes) (fields_autoplaced)
-    (property "Reference" "U?" (id 0) (at 227.33 23.5456 0))
-    (property "Value" "UPD301B/C" (id 1) (at 227.33 26.0856 0))
-    (property "Footprint" "" (id 2) (at 161.925 40.005 0)
+    (property "Reference" "U?" (id 0) (at 139.065 78.7906 0))
+    (property "Value" "UPD301B/C" (id 1) (at 139.065 81.3306 0))
+    (property "Footprint" "" (id 2) (at 73.66 95.25 0)
       (effects (font (size 1.27 1.27)) hide)
     )
-    (property "Datasheet" "" (id 3) (at 161.925 40.005 0)
+    (property "Datasheet" "" (id 3) (at 73.66 95.25 0)
       (effects (font (size 1.27 1.27)) hide)
     )

Commit message: updated
Parts:
- removed D?: RBR1VWM30ATFTR, ppse_2021:Package-PMDE, symbol Device:D_Schottky
- removed D?: ESD9B5.0ST5G, Diode_SMD:D_SOD-923, symbol Diode:ESD9B5.0ST5G
- removed P?: USB_C_Plug_USB2.0, symbol Connector:USB_C_Plug_USB2.0
- removed U?: UPD301B/C, symbol ICCI-LIB:UPD301B/C
- added C? (x3): 100n, symbol Device:C
- added C? (x3): 4.7u, symbol Device:C
- added D?: SD05_SOD323, Diode_SMD:D_SOD-323, symbol Diode:SD05_SOD323
- added D?: TX_LED, symbol Device:LED
- added D?: PRTR5V0U2AX,215, symbol ICCI-LIB:PRTR5V0U2AX,215
- added D?: RX_LED, symbol Device:LED
- added J?: USB_C_Receptacle_USB2.0, Connector_USB:USB_C_Receptacle_Amphenol_12401548E4-2A, symbol Connector:USB_C_Receptacle_USB2.0
- added JP?: SolderJumper_2_Open, symbol Jumper:SolderJumper_2_Open
- added Q? (x2): BC847, Package_TO_SOT_SMD:SOT-23, symbol Transistor_BJT:BC847
- added R? (x2): 10k, symbol Device:R
- added R? (x3): 1k, symbol Device:R
- added R?: 22.1k, symbol Device:R
- added R? (x2): 22R, symbol Device:R
- added R?: 47.5k, symbol Device:R
- added R?: 5.1k, symbol Device:R
Connections:
- net VBUS_FILTERED is gone; now on net VBUS: C?.1, C?.1, FB?.2
- net GND: now also U?.29 (GND), U?.3 (GND), C?.2, C?.2, C?.2, C?.2, C?.2, C?.2, D?.1, D?.1 (A1), J?.A1 (GND), J?.A12 (GND), J?.B1 (GND), J?.B12 (GND), JP?.1 (A), R?.2, R?.2
- net VBUS: now also C?.1, C?.1, D?.4, R?.1; no longer FB?.1
- net CC1: now reaches R?.1
- net CC1: now also J?.A5 (CC1)
- net CHREN: now reaches U?.13 (CHREN)
- net CHR1: now reaches U?.14 (CHR1)
- net CHR0: now reaches U?.15 (CHR0)
- net at U?.18 (~{RXT}/GPIO.1): now also D?.1 (K)
- net at U?.19 (~{TXT}/GPIO.0): now also D?.1 (K)
- net ~{RTS}: now reaches U?.24 (~{RTS})
- net ~{RTS}: now also Q?.2 (E), R?.1
- net TXD: now reaches U?.25 (RXD)
- net RXD: now reaches U?.26 (TXD)
- net ~{DTR}: now reaches U?.28 (~{DTR})
- net ~{DTR}: now also Q?.2 (E), R?.1
- net at U?.4 (D+): now also R?.2
- net at U?.5 (D-): now also R?.2
- net +3V3: now reaches U?.6 (VDD)
- net +3V3: now also U?.7 (VREGIN), C?.1, C?.1, C?.1, C?.1, R?.1, R?.1, R?.1
- net at U?.8 (VBUS): now also R?.1, R?.2
- net at U?.9 (~{RST}): now also R?.2
- new net: Q?.1 (B), R?.2 (x2)
- new net: J?.S1 (SHIELD), JP?.2 (B)
- new net: D?.2 (A), R?.2 (x2)
- new net CC2: J?.B5 (CC2), R?.1
- new net D+: D?.2, J?.A6 (D+), J?.B6 (D+), R?.1
- new net D-: D?.3, J?.A7 (D-), J?.B7 (D-), R?.1
- new net EN: Q?.3 (C)
- new net IO0: Q?.3 (C)
- new net VBUS_PRE: D?.2 (A2), FB?.1, J?.A4 (VBUS), J?.A9 (VBUS), J?.B4 (VBUS), J?.B9 (VBUS)
- no-connect marks 1 -> 13
Other:
- note added: "1.5A (and more?)"
- note added: "100mA"
- note added: "5.1k for 3A 5V device"
- note added: "500mA"
- note added: "Low Cap. ESD Protection"
- note added: "Test for best EMI solution"
- note added: "USB Type C"
- note removed: "5.1k for 3A 5V"
- note removed: "USB"
- note removed: "USB BC (Battery Charging) Standard coesistente con USB PD (Power Delivery) Permette di eccedere i 500mA in USB2.0 e 900mA in USB3.0 ed arrivare fino a 1.5A. NOTA: siccome i connettori USB supportano fino a 5A, alcuni produttori alzano la corrente fino a livelli più alti (tipo i classici 2A). Il dispositivo caricatore si identifica come tale segnalando l'assenza di dati nei segnali D+ e D- ponendo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"
- moved on the sheet: C?, FB?, R?, U?

Commit message: updated
Parts:
- removed JP?: SolderJumper_2_Open, symbol Jumper:SolderJumper_2_Open
- added R?: 0R, symbol Device:R
Connections:
- net GND: now also R?.1
- net at J?.S1 (SHIELD): now also R?.2
Changed lines of the file:
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@@
-    (pin "2")
-  )
-  (symbol (lib_id "Jumper:SolderJumper_2_Open") (at 42.545 118.11 90) (unit 1)
-    (in_bom yes) (on_board yes)
-    (property "Reference" "JP?" (id 0) (at 37.465 118.11 90)
-      (effects (font (size 1.27 1.27)) (justify right))
-    )
-    (property "Value" "SolderJumper_2_Open" (id 1) (at 45.085 119.3799 90)
-      (effects (font (size 1.27 1.27)) (justify right) hide)
-    )
-    (property "Footprint" "" (id 2) (at 42.545 118.11 0)
-      (effects (font (size 1.27 1.27)) hide)
-    )
-    (property "Datasheet" "~" (id 3) (at 42.545 118.11 0)
-      (effects (font (size 1.27 1.27)) hide)
-    )
-    (pin "1")
     (pin "2")
   )
@@
     (pin "1")
   )
+  (symbol (lib_id "Device:R") (at 42.545 118.11 180) (unit 1)
+    (in_bom no) (on_board yes)
+    (property "Reference" "R?" (id 0) (at 40.005 116.205 0))
+    (property "Value" "0R" (id 1) (at 40.005 118.11 0))
+    (property "Footprint" "" (id 2) (at 44.323 118.11 90)
+      (effects (font (size 1.27 1.27)) hide)
+    )
+    (property "Datasheet" "~" (id 3) (at 42.545 118.11 0)
+      (effects (font (size 1.27 1.27)) hide)
+    )
+    (property "Place" "DNP" (id 4) (at 39.37 120.015 0))
+    (pin "1")
+    (pin "2")
+  )
   (symbol (lib_id "Device:C") (at 107.95 71.12 0) (unit 1)
