File: ICCI-HW/Sensors.kicad_sch (KiCad schematic)
At the start: 19 parts, among them U301 DS18B20, U302 BH1750FVI-TR, U303 TCS34725FN, U304 TSL2561, U305 AS7341

Commit message: fw: updates
Parts:
- added C312, C313: 100n, Capacitor_SMD:C_0603_1608Metric, symbol Device:C
- added R304, R305: DNP, Resistor_SMD:R_0603_1608Metric, symbol Device:R
- added R306: 200k, Resistor_SMD:R_0603_1608Metric, symbol Device:R
- added U306: PCA9306GM,125, ICCI-LIB:PCA9306GM, symbol ICCI-LIB:PCA9306GM,125
- C305: renamed from C301; value 4,7u -> 4.7u
- renumbered C305 to C301, C310 to C306, C306 to C310, U305 to U302, U302 to U303, U303 to U304, U304 to U305
Connections:
- net +1V8: now also C312.1, R304.1, R305.1, U306.2 (VREF1)
- net +3V3: now also R306.1
- net GND: now also C312.2, C313.2, U306.1 (GND)
- net SCL0: now also U306.6 (SCL2); no longer U302.2 (SCL)
- net SDA0: now also U306.5 (SDA2); no longer U302.8 (SDA)
- new net: C313.1, R306.2, U306.7 (VREF2), U306.8 (EN)
- new net SCL0_1V8: R305.2, U302.2 (SCL), U306.3 (SCL1)
- new net SDA0_1V8: R304.2, U302.8 (SDA), U306.4 (SDA1)
Other:
- note added: "1V8 side should be as short as possible"
- note added: "DS report no pull-up, need testing."
- note added: "SDA, SCL, INT, LDR seems to be 3V3 tolerant but for reliability use level translator"
- note removed: "SDA, SCL, INT, LDR are 3V3 tolerant"
- moved on the sheet: C301, C302, C303, C304, C305, C306, C307, C308, C309, C310, C311, R301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
