File: ICCI-HW/ESP.kicad_sch (KiCad schematic)
At the start: 47 parts, among them J501 JTAG, SW501 SW_BOOT, SW502 SW_RST, SW503 SW_LOG_SD_EN, SW504 SW_RST_PROV, SW505 SW_RGB_CHRG, SW506 SW_SLEEP, U501 ESP32-WROVER-IE/E, U502 SX1503I091TRT

Commit message: fw: updates
Parts:
- removed R507, R508: 0R, Resistor_SMD:R_0603_1608Metric, symbol Device:R
- R501, R502, R503, R504: value 4.7k -> 2.2k
- TP501, TP502, TP503, TP504, TP505, TP506, TP507, TP508: now left out of the parts list
- renumbered R509 to R507, R510 to R508, R511 to R509, R512 to R510, R513 to R511, R514 to R512, R515 to R513, R516 to R514, R517 to R515
Connections:
- net Buzzer: now also U501.29 (IO5); no longer U502.13 (I/O[8])
- net GND: now also U501.39 (GND_PAD)
- net GPS_EXTINT: now also U502.20 (I/O[13])
- net GPS_TP: now also TP506.1, U502.23 (I/O[15])
- net ~{GPS_RESET}: now also U502.22 (I/O[14])
- net NINT renamed ~{EXP_INT}
- net NRESET renamed ~{EXP_RESET}
- new net ~{GPS_EN}: U502.13 (I/O[8])
- no-connect marks 11 -> 1
Other:
- note added: "Depending on the I2C bus speed, these values may be adjusted. 100KHz=4,7K 400KHz=2,2K In every case this need some testing."
- note added: "ESP Bootstrapping pins: MTDI (GPIO12) -> need to be kept low at startup: 0=LDO 3V3, 1=LDO 1V8 MTDO (GPIO15) -> 1=U0TXD Active 0=U0TXD Silent BOOT (GPIO0) -> 1=SPI, 0=Bootloader GPIO2 -> 0 for Bootloader mode GPIO5 (Pull-up at startup) SDIO timing Since we are not using SDIO interface we can freely use GPIO5."
- note added: "Internal pull-up"
- note added: "Up to 1.5A (more?)"
- note removed: "Depending on the I2C bus speed, these values may be decreased. 100KHz=4,7K 400KHz=2,2K"
- note removed: "ESP Bootstrapping pins: MTDI (GPIO12) -> need to be kept low at startup: 0=LDO 3V3, 1=LDO 1V8 MTDO (GPIO15) -> 1=U0TXD Active 0=U0TXD Silent BOOT (GPIO0) -> 1=SPI, 0=Bootloader GPIO2 -> 0 for Bootloader mode GPIO5 (Pull-up at startup) SDIO timing"
- note removed: "Up to 1.5A (and maybe more?)"
- moved on the sheet: R514, R515, TP506, U502

Commit message: hw: updates
Other:
- note added: "Show status on RGB Led (for 5s)"
- note removed: "Show charging status on RGB Led for 5s"
- company: tollsimy -> Simone Tollardo
Changed lines of the file:
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@@
   (title_block
     (title "ESP")
-    (date "2022-05-04")
+    (date "2022-07-14")
     (rev "BETA")
-    (company "tollsimy")
+    (company "Simone Tollardo")
   )
   (junction (at 210.82 55.245) (diameter 0) (color 0 0 0 0)
@@
     (stroke (width 0) (type default) (color 0 0 0 0))
   )
-  (wire (pts (xy 170.18 61.595) (xy 163.83 61.595))
+  (wire (pts (xy 172.72 61.595) (xy 163.83 61.595))
     (stroke (width 0) (type default) (color 0 0 0 0))
   )
@@
     (stroke (width 0) (type default) (color 0 0 0 0))
   )
+  (wire (pts (xy 31.115 180.34) (xy 36.195 180.34))
+    (stroke (width 0) (type default) (color 0 0 0 0))
+  )
   (wire (pts (xy 116.205 133.35) (xy 111.76 133.35))
     (stroke (width 0) (type default) (color 0 0 0 0))
@@
   )
   (wire (pts (xy 136.525 123.19) (xy 136.525 124.46))
-    (stroke (width 0) (type default) (color 0 0 0 0))
-  )
-  (wire (pts (xy 36.195 180.34) (xy 31.75 180.34))
     (stroke (width 0) (type default) (color 0 0 0 0))
   )
@@
     (effects (font (size 1.27 1.27)) (justify left bottom))
   )
-  (text "Show charging\nstatus on RGB \nLed for 5s" (at 149.225 162.56 0)
+  (text "Show status\non RGB Led\n(for 5s)" (at 149.225 162.56 0)
     (effects (font (size 1.27 1.27)) (justify left bottom))
   )
@@
     (effects (font (size 1.27 1.27)) (justify left))
   )
-  (hierarchical_label "IO0" (shape input) (at 170.18 61.595 0)
+  (hierarchical_label "IO0" (shape input) (at 172.72 61.595 0)
     (effects (font (size 1.27 1.27)) (justify left))
   )
@@
     (pin "2")
   )
+  (symbol (lib_id "power:+3V_VBAT") (at 31.115 180.34 0) (unit 1)
+    (in_bom yes) (on_board yes)
+    (property "Reference" "#PWR0116" (id 0) (at 31.115 184.15 0)
+      (effects (font (size 1.27 1.27)) hide)
+    )
+    (property "Value" "+3V_VBAT" (id 1) (at 31.115 176.53 0))
+    (property "Footprint" "" (id 2) (at 31.115 180.34 0)
+      (effects (font (size 1.27 1.27)) hide)
+    )
+    (property "Datasheet" "" (id 3) (at 31.115 180.34 0)
+      (effects (font (size 1.27 1.27)) hide)
+    )
+    (pin "1")
+  )
   (symbol (lib_id "power:+BATT") (at 17.78 174.625 0) (unit 1)
     (in_bom yes) (on_board yes)
@@
     (pin "1")
   )
-  (symbol (lib_name "ESP32-WROVER-IE{slash}E_1") (lib_id "ICCI-LIB:ESP32-WROVER-IE{slash}E") (at 143.51 51.435 0) (unit 1)
+  (symbol (lib_id "ICCI-LIB:ESP32-WROVER-IE{slash}E") (at 143.51 51.435 0) (unit 1)
     (in_bom yes) (on_board yes) (fields_autoplaced)
     (property "Reference" "U501" (id 0) (at 143.51 21.59 0))
@@
       (effects (font (size 1.27 1.27)) hide)
     )
-    (pin "1")
-  )
-  (symbol (lib_id "power:+3VBAT") (at 31.75 180.34 0) (unit 1)
-    (in_bom yes) (on_board yes)
-    (property "Reference" "#PWR0504" (id 0) (at 31.75 184.15 0)
-      (effects (font (size 1.27 1.27)) hide)
-    )
-    (property "Value" "3V_VBAT" (id 1) (at 31.75 176.53 0))
-    (property "Footprint" "" (id 2) (at 31.75 180.34 0)
-      (effects (font (size 1.27 1.27)) hide)
-    )
-    (property "Datasheet" "" (id 3) (at 31.75 180.34 0)
-      (effects (font (size 1.27 1.27)) hide)
-    )
