File: ICCI-HW/ICCI-HW.kicad_pcb (KiCad board)
At the start: 4 copper layers, 100 x 100 mm, 200 parts, among them J201 USB_C_Receptacle_USB2.0, J401 EXP0, J402 EXP1, J403 DM3AT-SF-PEJM5, J501 JTAG, Q201 PDTC114Y, Q202 PDTC114Y, Q203 NX7002AK, Q401 RZM001P02, Q402 PDTC114Y, Q403 PDTC114Y, Q404 PDTC114Y, Q405 PDTC114Y, SW501 SW_BOOT, SW502 SW_RST, SW503 SW_LOG_SD_EN, SW504 SW_RST_PROV, SW505 SW_RGB_CHRG, SW506 SW_SLEEP, SW601 SW_SPDT, U201 CP2102N-Axx-xQFN28, U301 DS18B20, U302 AS7341, U303 BH1750FVI-TR, U304 TCS34725FN, U305 TSL2561, U306 PCA9306GM,125, U401 PCF2127AT, U402 SAM-M8Q, U501 ESP32-WROVER-IE/E, U502 SX1503I091TRT, U601 NCV8164ASN180T1G, U602 AP62301WU-7, U603 MAX77960BEFV12+

Commit message: start layout
Parts:
- removed J402: EXP1, Connector_PinHeader_2.54mm:PinHeader_1x04_P2.54mm_Vertical
- removed NT201: NetTie_2, NetTie:NetTie-2_SMD_Pad0.5mm
- removed TP506: TP_CLK/TP, TestPoint:TestPoint_Plated_Hole_D2.0mm
- added JP501: SolderJumper_3_Bridged12, Jumper:SolderJumper-3_P1.3mm_Open_RoundedPad1.0x1.5mm_NumberLabels, F.Cu at (48.9, 109.6)
- added JP502: SolderJumper_3_Bridged12, Jumper:SolderJumper-3_P1.3mm_Open_RoundedPad1.0x1.5mm_NumberLabels, F.Cu at (43.6, 109.6)
- added JP503: SolderJumper_3_Bridged12, Jumper:SolderJumper-3_P1.3mm_Open_RoundedPad1.0x1.5mm_NumberLabels, F.Cu at (46.2, 109.6)
- added Q204: NX7002AK, Package_TO_SOT_SMD:SOT-23, F.Cu at (88.2, 148.7)
- J401: value EXP0 -> EXP; footprint Connector_PinHeader_2.54mm:PinHeader_1x04_P2.54mm_Vertical -> Connector_PinSocket_2.54mm:PinSocket_2x03_P2.54mm_Horizontal
- J501: footprint Connector_PinHeader_2.54mm:PinHeader_1x04_P2.54mm_Vertical -> ICCI-LIB:JST_B6B-XH-A
- TP501, TP502, TP503, TP504, TP505, TP507, TP508: footprint TestPoint:TestPoint_Plated_Hole_D2.0mm -> TestPoint:TestPoint_THTPad_D1.5mm_Drill0.7mm
- U301: footprint Package_TO_SOT_THT:TO-92_Inline -> ICCI-LIB:DS18B20 Hor.; moved to F.Cu
- moved TP504 125.7 mm to (69.2, 155.2)
- moved TP505 120.0 mm to (44.9, 126.8)
- moved TP502 114.0 mm to (97.2, 159.7)
- moved C313 103.5 mm to (98.9, 114.2), turned to 90 degrees
- moved R302 103.4 mm to (92.7, 117.7), turned to -90 degrees
- moved R303 103.3 mm to (86.9, 124.8)
- moved R306 102.2 mm to (97.3, 116.9), turned to 90 degrees
- moved TP507 101.9 mm to (83.7, 145.2)
- moved R305 98.3 mm to (94.7, 112.6), turned to -90 degrees
- moved C304 97.9 mm to (85.0, 118.2), turned to -90 degrees
- moved C312 97.2 mm to (97.0, 111.8)
- moved C303 95.4 mm to (88.3, 114.2), turned to -90 degrees
- moved U306 95.4 mm to (96.8, 114.0), turned to -90 degrees
- moved R304 94.9 mm to (93.1, 113.5), turned to -90 degrees
- moved C311 94.5 mm to (87.3, 117.5)
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Connections:
- net Net-(BT601-PadC1+) renamed /BATT + POWER/B1-B2
- D605 pad 1: VCC -> /BATT + POWER/SYS
- D605 pad 2: +BATT -> /BATT + POWER/BATT
- J401 pad 1: +3V3 -> GND
- J401 pad 2: /AUX + Peripherals/SCL0 -> /AUX + Peripherals/SDA1
- J401 pad 3: /AUX + Peripherals/SDA0 -> /AUX + Peripherals/SCL1
- J401 pad 4: GND -> /AUX + Peripherals/SDA0
- J501 pad 1: /ESP/TMS -> GND
- J501 pad 3: /ESP/TCK -> /ESP/TDO
- J501 pad 4: /ESP/TDO -> /ESP/TCK
- R403 pad 2: /AUX + Peripherals/~{GPS_RESET} -> /AUX + Peripherals/~{RTC_RST}
- R405 pad 2: /AUX + Peripherals/GPS_TP -> /AUX + Peripherals/RTC_CLKOUT
- R406 pad 2: /AUX + Peripherals/GPS_EXTINT -> /AUX + Peripherals/~{RTC_INT}
- RN401 pad 1: /AUX + Peripherals/SD_DET_B -> /AUX + Peripherals/~{SD_DET}
- U401 pad 16: /AUX + Peripherals/~{GPS_RESET} -> /AUX + Peripherals/~{RTC_RST}
- U401 pad 17: /AUX + Peripherals/GPS_EXTINT -> /AUX + Peripherals/~{RTC_INT}
- U401 pad 7: /AUX + Peripherals/GPS_TP -> /AUX + Peripherals/RTC_CLKOUT
- U502 pad 20: /AUX + Peripherals/GPS_EXTINT -> Net-(JP503-Pad2)
- U502 pad 22: /AUX + Peripherals/~{GPS_RESET} -> Net-(JP502-Pad2)
- U502 pad 23: /AUX + Peripherals/GPS_TP -> Net-(JP501-Pad2)
Routing:
- net /USB/D+: track 0.00 -> 36.8 mm, vias 0 -> 1
- net /USB/D-: track 0.00 -> 35.7 mm, vias 0 -> 1
- net /BATT + POWER/PVL: track 0.00 -> 25.6 mm, vias 0 -> 3
- net Net-(J201-PadS1): track 0.00 -> 24.4 mm
- net VBUS: track 0.00 -> 21.1 mm, vias 0 -> 3
- net /BATT + POWER/VSET: track 0.00 -> 16.0 mm
- net /USB/CC2: track 0.00 -> 15.2 mm, vias 0 -> 1
- net /USB/CC1: track 0.00 -> 11.6 mm
- net /BATT + POWER/ITO: track 0.00 -> 11.4 mm
- net /BATT + POWER/INLIM: track 0.00 -> 10.4 mm
- net /BATT + POWER/ISET_R: track 0.00 -> 10.2 mm, vias 0 -> 2
- net GND: track 0.00 -> 9.80 mm, vias 0 -> 27
- net /BATT + POWER/ISET: track 0.00 -> 5.75 mm
- net /ESP/RXDR: track 0.00 -> 4.33 mm
- net /BATT + POWER/SYSA: track 0.00 -> 4.31 mm
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- added copper zone on In2.Cu, net +3V3
- added copper zone on B.Cu, net /BATT + POWER/B1-B2
- added copper zone on B.Cu, net GND
- added copper zone on F.Cu, net GND
- added copper zone on In1.Cu, net GND
Other:
- board text added: "Aperture"
- board text added: "CAUTION, DO NOT INSERT BATTERY UPSIDE DOWN!"
- board text added: "Diffuser"
- board text added: "W: 3V3 Only!"
- board text removed: "How to handle alternate versions?"
- board text removed: "Lens"
- board text removed: "Se utilizzo l'altra versione con più sensori forse la lente convessa non va bene perchè non si riescono a sovrapporre più di tanto"
- board text removed: "TODO: add programming UART interface as well as debug jtag interface with appropriate headers"
- board text removed: "WARNING, DO NOT INSERT BATTERY UPSIDE DOWN!"

Commit message: layout updates
Parts:
- J401: footprint Connector_PinSocket_2.54mm:PinSocket_2x03_P2.54mm_Horizontal -> Connector_PinSocket_2.54mm:PinSocket_2x02_P2.54mm_Horizontal
- moved R623 16.6 mm to (60.8, 140.8), turned to -90 degrees
- moved C406 16.1 mm to (53.4, 146.9), turned to -145 degrees
- moved D402 8.72 mm to (118.4, 98.0), turned to -90 degrees
- moved C409 8.61 mm to (119.6, 102.0), turned to 90 degrees
- moved R615 8.13 mm to (61.3, 111.8), turned to 180 degrees
- moved R616 6.91 mm to (69.5, 152.2), turned to 0 degrees
- moved TP501 6.62 mm to (64.8, 112.3)
- moved C410 5.86 mm to (118.1, 102.0), turned to 90 degrees
- moved D604 4.83 mm to (61.1, 113.6), turned to 180 degrees
- moved RN401 3.27 mm to (110.0, 109.1), turned to -90 degrees
- moved C608 2.57 mm to (67.6, 130.5), turned to 0 degrees
- moved R405 1.95 mm to (56.2, 145.1), turned to 125 degrees
- moved U602 1.90 mm to (69.0, 127.5)
- moved R617 1.79 mm to (61.8, 118.1), turned to 0 degrees
- moved JP501 1.73 mm to (48.2, 111.2)
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Connections:
- net Net-(C311-Pad1) renamed /Sensors/DVI
- net Net-(D602-Pad1) renamed /BATT + POWER/FUSE_OUT
- net Net-(R302-Pad1) renamed /Sensors/ADDR
- net Net-(SW601-Pad2) renamed /BATT + POWER/EN
- D605 pad 1: /BATT + POWER/SYS -> VCC
- D605 pad 2: /BATT + POWER/BATT -> +BATT
- J401 pad 2: /AUX + Peripherals/SDA1 -> /AUX + Peripherals/SDA0
- J401 pad 3: /AUX + Peripherals/SCL1 -> /AUX + Peripherals/SCL0
- J401 pad 4: /AUX + Peripherals/SDA0 -> +3V3
Routing:
- net /AUX + Peripherals/SCL1: track 0.00 -> 183.6 mm, vias 0 -> 7
- net /AUX + Peripherals/SDA1: track 0.00 -> 177.5 mm, vias 0 -> 4
- net GND: track 9.80 -> 184.1 mm, vias 27 -> 166
- net /ESP/SLEEP: track 0.00 -> 89.9 mm, vias 0 -> 2
- net /AUX + Peripherals/SDA0: track 0.00 -> 83.5 mm, vias 0 -> 4
- net /AUX + Peripherals/SCL0: track 0.00 -> 83.0 mm, vias 0 -> 4
- net Net-(JP503-Pad2): track 0.00 -> 80.6 mm, vias 0 -> 2
- net +3V3: track 0.00 -> 74.3 mm, vias 0 -> 63
- net Net-(JP502-Pad2): track 0.00 -> 73.6 mm, vias 0 -> 2
- net VCC: track 0.00 -> 69.1 mm, vias 0 -> 45
- net Net-(JP501-Pad2): track 0.00 -> 64.5 mm, vias 0 -> 2
- net /AUX + Peripherals/~{SD_CS}: track 0.00 -> 64.3 mm, vias 0 -> 2
- net /AUX + Peripherals/VSPI_MOSI: track 0.00 -> 62.0 mm, vias 0 -> 2
- net /AUX + Peripherals/RTC_CLKOUT: track 0.00 -> 53.4 mm, vias 0 -> 4
- net /AUX + Peripherals/VSPI_MISO: track 0.00 -> 52.1 mm, vias 0 -> 2
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- added copper zone on B.Cu, net +3V3
- added copper zone on F.Cu, net +3V3
- added copper zone on B.Cu, net +BATT
- added copper zone on F.Cu, net +BATT
- added copper zone on F.Cu, net /BATT + POWER/BST1
- added copper zone on B.Cu, net /BATT + POWER/CHGIN
- added copper zone on F.Cu, net /BATT + POWER/CHGIN
- added copper zone on B.Cu, net /BATT + POWER/FUSE_OUT
- added copper zone on F.Cu, net /BATT + POWER/FUSE_OUT
- added copper zone on B.Cu, net /BATT + POWER/LX1
- added copper zone on F.Cu, net /BATT + POWER/LX1
- added copper zone on B.Cu, net /BATT + POWER/LX2
- added copper zone on F.Cu, net /BATT + POWER/LX2
- added copper zone on F.Cu, net /BATT + POWER/SW_FB
- added copper zone on F.Cu, net /BATT + POWER/SW_NODE
- added copper zone on F.Cu, net /BATT + POWER/SW_NODE_OUT
- added copper zone on B.Cu, net VCC
- added copper zone on F.Cu, net VCC
Other:
- board text added: "Questione GND Planes"
- board text added: "TVS"
