File: ICCI-HW/ICCI-HW.kicad_pcb (KiCad board)
At the start: 4 copper layers, 100 x 100 mm, 201 parts, among them J201 USB_C_Receptacle_USB2.0, J401 EXP, J403 DM3AT-SF-PEJM5, J501 JTAG, Q201 PDTC114Y, Q202 PDTC114Y, Q203 NX7002AK, Q204 NX7002AK, Q401 RZM001P02, Q402 PDTC114Y, Q403 PDTC114Y, Q404 PDTC114Y, Q405 PDTC114Y, SW501 SW_BOOT, SW502 SW_RST, SW503 SW_LOG_SD_EN, SW504 SW_RST_PROV, SW505 SW_RGB_CHRG, SW506 SW_SLEEP, SW601 SW_SPDT, U201 CP2102N-Axx-xQFN28, U301 DS18B20, U302 AS7341, U303 BH1750FVI-TR, U304 TCS34725FN, U305 TSL2561, U306 PCA9306GM,125, U401 PCF2127AT, U402 SAM-M8Q, U501 ESP32-WROVER-IE/E, U502 SX1503I091TRT, U601 NCV8164ASN180T1G, U602 AP62301WU-7, U603 MAX77960BEFV12+

Commit message: layout updates
Parts:
- moved D604 44.2 mm to (65.9, 157.5)
- moved R615 44.2 mm to (66.1, 155.8)
- moved R301 11.4 mm to (89.3, 124.1), turned to 90 degrees
- moved C305 9.51 mm to (86.2, 124.1), turned to 90 degrees
- moved TP501 8.35 mm to (70.8, 118.0)
- moved C310 8.02 mm to (87.8, 124.1), turned to 90 degrees
- moved R303 4.44 mm to (90.0, 121.7), turned to 180 degrees
- moved R506 3.18 mm to (93.0, 126.0), turned to -90 degrees
- moved R505 3.06 mm to (91.5, 126.0), turned to 90 degrees
- moved R511 1.08 mm to (104.7, 145.0)
- moved R512 0.96 mm to (100.7, 141.6)
- moved TP504 0.93 mm to (70.1, 155.2)
- moved C515 0.57 mm to (101.8, 112.4)
- moved C513 0.56 mm to (101.8, 114.0)
- moved R209 0.53 mm to (103.2, 147.2)
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Routing:
- net /BATT + POWER/MAX_INOKB: track 5.31 -> 134.0 mm, vias 0 -> 4
- net /BATT + POWER/MAX_INTB: track 4.65 -> 108.1 mm, vias 0 -> 4
- net /ESP/EN: track 36.2 -> 127.9 mm, vias 2 -> 5
- net /ESP/IO0: track 6.01 -> 93.8 mm, vias 0 -> 4
- net /ESP/Buzzer: track 0.00 -> 59.2 mm
- net +3V0: track 36.9 -> 90.7 mm, vias 2 -> 5
- net /USB/CHREN: track 0.00 -> 47.1 mm, vias 0 -> 4
- net /USB/CHR0: track 0.00 -> 44.7 mm, vias 0 -> 2
- net GND: track 184.1 -> 226.5 mm, vias 166 -> 200
- net /USB/CHR1: track 0.00 -> 42.0 mm, vias 0 -> 2
- net /AUX + Peripherals/GPS_VCC: track 0.00 -> 39.1 mm, vias 0 -> 2
- net +3V3: track 74.3 -> 112.8 mm, vias 63 -> 71
- net Net-(Q203-Pad1): track 5.21 -> 43.0 mm, vias 2 -> 3
- net /ESP/DS_DQ: track 0.00 -> 36.3 mm, vias 0 -> 2
- net /AUX + Peripherals/GPS_TP: track 33.6 -> 57.2 mm, vias 2 -> 4
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- added copper zone on B.Cu, net /BATT + POWER/BST1
- added copper zone on In2.Cu, net GND
Other:
- board text added: "Antenna ESP deve andare fuori pcb, come fare? tagliarla?"
- board text added: "Bug GND vias connessi al plane interno 2 (3V3) sotto ESP EPAD"
- board text added: "Completely reset DRC exlusion (courtryard overlap, silkscreen etc) and redo"
- board text added: "General Check + Check planes separately"
- board text added: "Pour anche su TOP e BOTTOM?"
- board text added: "Rivisitare GPS layout secondo DS"
